File: inside/inside.kicad_pcb (KiCad board)
At the start: 2 copper layers, 7 parts, among them J1 Barrel_Jack, J2 Conn_01x04, J3 Conn_01x04, J4 Conn_01x04, U2 ESP32-WROOM-32

Commit message: finished pcb
Parts:
- removed J2, J3, J4: Conn_01x04, Converter_DCDC:buck voltage converter
- added J5: Conn_01x03, custom:1~5PCS EGBO DD4012SA 24v-12v, F.Cu at (127.2, 82.5)
- moved J1 68.9 mm to (100.3, 75.1), turned to -90 degrees
- moved A3 52.5 mm to (153.8, 111.4), turned to 180 degrees
- moved A2 49.9 mm to (101.2, 92.3)
- moved U2 32.6 mm to (127.5, 104.8)
Connections:
- A2 pad 3: unconnected-(A2-1B-Pad3) -> Net-(A2-1B)
- A2 pad 4: unconnected-(A2-1A-Pad4) -> Net-(A2-1A)
- A2 pad 5: unconnected-(A2-2A-Pad5) -> Net-(A2-2A)
- A2 pad 6: unconnected-(A2-2B-Pad6) -> Net-(A2-2B)
- A3 pad 2: Net-(A3-VDD) -> Net-(A2-VDD)
- A3 pad 3: unconnected-(A3-1B-Pad3) -> Net-(A3-1B)
- A3 pad 4: unconnected-(A3-1A-Pad4) -> Net-(A3-1A)
- A3 pad 5: unconnected-(A3-2A-Pad5) -> Net-(A3-2A)
- A3 pad 6: unconnected-(A3-2B-Pad6) -> Net-(A3-2B)
- U2 pad 2: Net-(J2-Pin_4) -> Net-(A2-VDD)
Routing:
- net GND: track 0.00 -> 152.0 mm, vias 0 -> 4
- net Net-(A2-VMOT): track 0.00 -> 125.7 mm
- net Net-(A2-VDD): track 0.00 -> 95.0 mm
- net Net-(A3-DIR): track 0.00 -> 25.4 mm, vias 0 -> 1
- net Net-(A3-STEP): track 0.00 -> 24.9 mm, vias 0 -> 1
- net Net-(A2-DIR): track 0.00 -> 11.0 mm
- net Net-(A2-STEP): track 0.00 -> 6.63 mm
- added copper zone on B.Cu, net GND
- added copper zone on F.Cu, net GND
Other:
- board outline added: 88.6 x 78.2 mm
- board text added: "love lola 2025"
