File: inside/inside.kicad_sch (KiCad schematic)
At the start: 7 parts, among them J1 Barrel_Jack, U1 TSR_1-2433, U2 ESP32-WROOM-32, U4 TSR_1-2433, U5 TSR_1-2433

Commit message: svgs made
Parts:
- removed U1, U4, U5: TSR_1-2433, Converter_DCDC:Converter_DCDC_TRACO_TSR-1_THT, symbol Regulator_Switching:TSR_1-2433
- added J2, J3, J4: Conn_01x04, Converter_DCDC:buck voltage converter, symbol Connector_Generic:Conn_01x04
- added bvc1, bvc2: ~, symbol Converter_DCDC:buck_voltage_converter
- J1: footprint (none) -> Connector_BarrelJack:BarrelJack_Horizontal
Connections:
- net GND: now also J2.2 (Pin_2), J2.3 (Pin_3), J3.2 (Pin_2), J3.3 (Pin_3), J4.2 (Pin_2), J4.3 (Pin_3)
- net at A3.2 (VDD): now also J4.4 (Pin_4)
- net at A2.8 (VMOT), A3.8 (VMOT), J1.1: now also J2.1 (Pin_1), J3.1 (Pin_1), J4.1 (Pin_1)
- net at A2.2 (VDD): now also J3.4 (Pin_4)
- net at U2.2 (VDD): now also J2.4 (Pin_4)

Commit message: finished pcb
Parts:
- removed J2, J3, J4: Conn_01x04, Converter_DCDC:buck voltage converter, symbol Connector_Generic:Conn_01x04
- removed bvc1, bvc2: ~, symbol Converter_DCDC:buck_voltage_converter
- added J2, J3: Conn_01x04_Pin, Connector_PinHeader_1.00mm:PinHeader_1x04_P1.00mm_Vertical, symbol Connector:Conn_01x04_Pin
- added J5: Conn_01x03, custom:1~5PCS EGBO DD4012SA 24v-12v, symbol Connector_Generic:Conn_01x03
Connections:
- net GND: now also J5.2 (Pin_2)
- net at A2.8 (VMOT), A3.8 (VMOT), J1.1: now also J5.3 (Pin_3)
- net at A2.2 (VDD): now also A3.2 (VDD), U2.2 (VDD), J5.1 (Pin_1)
- net at A3.3 (1B): now also J2.4 (Pin_4)
- net at A3.4 (1A): now also J2.3 (Pin_3)
- net at A3.5 (2A): now also J2.2 (Pin_2)
- net at A3.6 (2B): now also J2.1 (Pin_1)
- net at A2.3 (1B): now also J3.4 (Pin_4)
- net at A2.4 (1A): now also J3.3 (Pin_3)
- net at A2.5 (2A): now also J3.2 (Pin_2)
- net at A2.6 (2B): now also J3.1 (Pin_1)
